File: Florian_PCB/LESR_MainBoard/Design_Files/LESR_MainBoard/LESR_MainBoard.sch (EAGLE design)
At the start: 46 parts, among them Q1 SS8050-G, Q2 SS8050-G, U1 TCA9548APWR, U2 NCP1117ST33T3G, U3 ESP32-WROOM-32, U4 CP2102N-A01-GQFN28, U5 SP0503BAHT

Commit message: JST Updated in Main B
Parts:
- removed LESR1, LESR2, LESR3, LESR4, LESR5, LESR6, LESR7, LESR8, SENSOR1, SENSOR2, SENSOR3, SENSOR4, SENSOR5, SENSOR6, SENSOR7, SENSOR8: Vertical Qwiic Connector, SparkFun-Connectors:QWIIC_CONNECTOR
- added CONN1, CONN2, CONN3, CONN4, CONN5, CONN6, CONN7, CONN8: JST_6_PIN_VERTICAL, SparkFun-Connectors:JST_6_PIN_VERTICAL
- added J1: DCJ0202, con-jack:DCJ0202
Connections:
- new net VIN: C1.1, CONN1.1, CONN1.5, CONN2.1, CONN2.5, CONN3.1, CONN3.5, CONN4.1, CONN4.5, CONN5.1, CONN5.5, CONN6.1, CONN6.5, CONN7.1, CONN7.5, CONN8.1, CONN8.5, J1.1, JP1.1, JP2.1, JP4.1, U2.IN
- net GND: now also CONN1.6, CONN2.6, CONN3.6, CONN4.6, CONN5.6, CONN6.6, CONN7.6, CONN8.6, J1.2, J1.3; no longer SENSOR1.1, SENSOR2.1, SENSOR3.1, SENSOR4.1, SENSOR5.1, SENSOR6.1, SENSOR7.1, SENSOR8.1
- net IO16: now also CONN7.4; no longer LESR7.3
- net IO17: now also CONN8.4; no longer LESR8.3
- net IO23: now also CONN1.4; no longer LESR1.3
- net IO25: now also CONN2.4; no longer LESR2.3
- net IO26: now also CONN3.4; no longer LESR3.3
- net IO27: now also CONN4.4; no longer LESR4.3
- net IO32: now also CONN5.4; no longer LESR5.3
- net IO33: now also CONN6.4; no longer LESR6.3
- net SC0: now also CONN1.2; no longer SENSOR1.4
- net SC1: now also CONN2.2; no longer SENSOR2.4
- net SC2: now also CONN3.2; no longer SENSOR3.4
- net SC3: now also CONN4.2; no longer SENSOR4.4
- net SC4: now also CONN5.2; no longer SENSOR5.4
- net SC5: now also CONN6.2; no longer SENSOR6.4
- net SC6: now also CONN7.2; no longer SENSOR7.4
- net SC7: now also CONN8.2; no longer SENSOR8.4
- net SD0: now also CONN1.3; no longer SENSOR1.3
- net SD1: now also CONN2.3; no longer SENSOR2.3
- net SD2: now also CONN3.3; no longer SENSOR3.3
- net SD3: now also CONN4.3; no longer SENSOR4.3
- net SD4: now also CONN5.3; no longer SENSOR5.3
- net SD5: now also CONN6.3; no longer SENSOR6.3
- net SD6: now also CONN7.3; no longer SENSOR7.3
- net SD7: now also CONN8.3; no longer SENSOR8.3
- net VBUS: no longer C1.1, JP1.1, JP2.1, JP4.1, SENSOR1.2, SENSOR2.2, SENSOR3.2, SENSOR4.2, SENSOR5.2, SENSOR6.2, SENSOR7.2, SENSOR8.2, U2.IN
Other:
- note added: "Connectors for LESR and Sensor"
- note removed: "ESP32 to LESR Ring"
- note removed: "ESP32 to Sensor Connectors"
